File: hardware/slice_template.kicad_sch (KiCad schematic)
At the start: 19 parts, among them J1 Conn_01x10_Socket, SW1 SW_DIP_x04, U1 AP63205

Commit message: did schematic
Parts:
- renumbered A2 to A1, J1 to J2, SW1 to SW2
Changed lines of the file:
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@@
 		(dnp no)
 		(fields_autoplaced yes)
-		(property "Reference" "A2"
+		(property "Reference" "A1"
 			(at 291.7033 156.21 0)
 			(effects
@@
 			(project ""
 				(path "/66043bca-a260-4915-9fce-8a51d324c687/a4d66d05-b498-454f-8d54-68b671c284b9"
-					(reference "A2")
+					(reference "A1")
 					(unit 1)
 				)
@@
 		(on_board yes)
 		(dnp no)
-		(property "Reference" "SW1"
+		(property "Reference" "SW2"
 			(at 201.93 114.554 0)
 			(effects
@@
 			(project "BREAD_Slice"
 				(path "/66043bca-a260-4915-9fce-8a51d324c687/a4d66d05-b498-454f-8d54-68b671c284b9"
-					(reference "SW1")
+					(reference "SW2")
 					(unit 1)
 				)
@@
 		(on_board yes)
 		(dnp no)
-		(property "Reference" "J1"
+		(property "Reference" "J2"
 			(at 65.532 120.142 0)
 			(effects
@@
 			(project ""
 				(path "/66043bca-a260-4915-9fce-8a51d324c687/a4d66d05-b498-454f-8d54-68b671c284b9"
-					(reference "J1")
-					(unit 1)
-				)
+					(reference "J2")
+					(unit 1)
+				)
