File: hardware/BREAD_Slice.kicad_pcb (KiCad board)
At the start: 4 copper layers, 100 x 145 mm, 26 parts, among them J1 Screw_Terminal_01x02, J2 Conn_01x10_Socket, J3 PCIE-036-02-X-D-TH, J4 PCIE-036-02-X-D-TH, J5 PCIE-036-02-X-D-TH, J6 PCIE-036-02-X-D-TH, SW2 SW_DIP_x04, U1 AP63205

Commit message: fix(hw): re-point stale library nicknames
These parts exist in KiCad-Master-Lib; the boards referenced libraries that no
longer exist (kml-custom, KML-Custom, and SparkFun libraries that never
contained the part) or names the library has since changed.

KiCad embeds footprint geometry in the .kicad_pcb, so the boards rendered and
fabricated correctly and the rot stayed invisible -- it only surfaces on
update-from-library, or when a generator tries to resolve a nickname.

Nickname/name only. No geometry is changed:

  KMLib_Mounting:Thermal Pad -> KMLib_Mounting:Thermal_Pad
  SparkFun-LED:WS2812-5050-4PIN -> KMLib_IC_SMD:WS2812-5050-4PIN
  kml-custom:AP63205WU-7 -> KMLib_IC_Power:AP63205WU-7_Buck_Regulator
  kml-custom:SOIC_05WU-7_DIO -> KMLib_IC_SMD:SOIC_05WU-7_DIO
  kml-custom:WS2812B_5050 -> SparkFun-LED:WS2812B_5050

Only references that failed to resolve were touched. Generic parts (<=4 pins)
and KiCad *-rescue libraries are deliberately excluded: fingerprint matching
cannot distinguish a 2-pin resistor from a 2-pin capacitor, so those are being
done by hand.
Parts:
- HS1: footprint KMLib_Mounting:Thermal Pad -> KMLib_Mounting:Thermal_Pad
Changed lines of the file:
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@@
 		)
 	)
-	(footprint "KMLib_Mounting:Thermal Pad"
+	(footprint "KMLib_Mounting:Thermal_Pad"
 		(layer "F.Cu")
 		(at 99.85 143.355)
